File: kicad/e-p-wifi-shield/e-p-wifi.sch (KiCad schematic (older format))
At the start: 33 parts, among them J2 T1, J3 Masse, J4 T2, SW1 ON/OFF, SW2 StSp, SW3 Sleep, U1 Arduino_MKR_WIFI_1010

Commit message: Maj du 5 novembre 2019
Parts:
- removed BT1: Battery_Cell, symbol Device:Battery_Cell
- removed J?: Conn_01x08-a, symbol e-p-wifi-rescue:Conn_01x08-a
- removed U1: Arduino_MKR_WIFI_1010, symbol e-p-wifi-rescue:Arduino_MKR_WIFI_1010-MCU_Module
- added J4: Conn_02x14_MKR1010, PinSocket_2x14_P2.54mm_Vertical, symbol e-p-wifi-rescue:Conn_02x14_MKR1010
- C1: footprint (none) -> Capacitor_THT:CP_Radial_D5.0mm_P2.50mm
- D1: footprint (none) -> LED_THT:LED_D3.0mm
- D2: renamed from D3; footprint (none) -> LED_THT:LED_D3.0mm
- D3: renamed from D4; footprint (none) -> LED_THT:LED_D3.0mm
- D4: renamed from D5; footprint (none) -> LED_THT:LED_D3.0mm
- D5: renamed from D2; footprint (none) -> LED_THT:LED_D3.0mm
- R1, R14, R7: footprint (none) -> Resistor_THT:R_Axial_DIN0207_L6.3mm_D2.5mm_P7.62mm_Horizontal
- R10: renamed from R13; footprint (none) -> Resistor_THT:R_Axial_DIN0207_L6.3mm_D2.5mm_P7.62mm_Horizontal
- R11: renamed from R8; footprint (none) -> Resistor_THT:R_Axial_DIN0207_L6.3mm_D2.5mm_P7.62mm_Horizontal
- R12: renamed from R10; footprint (none) -> Resistor_THT:R_Axial_DIN0207_L6.3mm_D2.5mm_P7.62mm_Horizontal
- R13: renamed from R12; footprint (none) -> Resistor_THT:R_Axial_DIN0207_L6.3mm_D2.5mm_P7.62mm_Horizontal
- R15: renamed from R16; footprint (none) -> Resistor_THT:R_Axial_DIN0207_L6.3mm_D2.5mm_P7.62mm_Horizontal
- R16: renamed from R17; footprint (none) -> Resistor_THT:R_Axial_DIN0207_L6.3mm_D2.5mm_P7.62mm_Horizontal
- R17: renamed from R18; footprint (none) -> Resistor_THT:R_Axial_DIN0207_L6.3mm_D2.5mm_P7.62mm_Horizontal
- R18: renamed from R15; footprint (none) -> Resistor_THT:R_Axial_DIN0207_L6.3mm_D2.5mm_P7.62mm_Horizontal
- R2: renamed from R4; footprint (none) -> Resistor_THT:R_Axial_DIN0207_L6.3mm_D2.5mm_P7.62mm_Horizontal
- R3: renamed from R5; footprint (none) -> Resistor_THT:R_Axial_DIN0207_L6.3mm_D2.5mm_P7.62mm_Horizontal
- R4: renamed from R2; footprint (none) -> Resistor_THT:R_Axial_DIN0207_L6.3mm_D2.5mm_P7.62mm_Horizontal
- R5: renamed from R3; footprint (none) -> Resistor_THT:R_Axial_DIN0207_L6.3mm_D2.5mm_P7.62mm_Horizontal
- R6: renamed from R1; footprint (none) -> Resistor_THT:R_Axial_DIN0207_L6.3mm_D2.5mm_P7.62mm_Horizontal
- R8: renamed from R9; footprint (none) -> Resistor_THT:R_Axial_DIN0207_L6.3mm_D2.5mm_P7.62mm_Horizontal
- R9: renamed from R11; footprint (none) -> Resistor_THT:R_Axial_DIN0207_L6.3mm_D2.5mm_P7.62mm_Horizontal
- SW1: value ON/OFF -> Conrad 711771
- renumbered J2 to J1, J3 to J2, J4 to J3
Connections:
- wire segments 120 -> 112
- no-connect marks 14 -> 13
Other:
- note removed: "+"
- note removed: "-"
- note removed: "Breadboard [3b]"
- note removed: "DS18B20"
- note removed: "Entretoise de fixation [16]"
- note removed: "[17]"
- note removed: "[4]"
- note removed: "[7]"
- moved on the sheet: D2, D3, D4, D5, R15, R16, R17, R18

Commit message: Maj du 07 novembre 2019
Parts:
- removed J1: T1, symbol Connector:Conn_01x03_Male
- removed J2: Masse, symbol Connector:Conn_01x01_Male
- removed J3: T2, symbol Connector:Conn_01x03_Male
- removed R1: 1 Ohm, Resistor_THT:R_Axial_DIN0207_L6.3mm_D2.5mm_P7.62mm_Horizontal, symbol Device:R
- added J1: Shunt, Connector_PinHeader_2.54mm:PinHeader_1x02_P2.54mm_Vertical, symbol Connector_Generic:Conn_01x02
- added J2: Vbat1, Connector_PinHeader_2.54mm:PinHeader_1x02_P2.54mm_Vertical, symbol Connector_Generic:Conn_01x02
- added J3: Masse T1, Connector_PinHeader_2.54mm:PinHeader_1x02_P2.54mm_Vertical, symbol Connector_Generic:Conn_01x02
- added J4: Température, Connector_PinHeader_1.00mm:PinHeader_1x06_P1.00mm_Vertical, symbol Connector_Generic:Conn_01x06
- added J5: Vbat2, Connector_PinHeader_2.54mm:PinHeader_1x02_P2.54mm_Vertical, symbol Connector_Generic:Conn_01x02
- J6: renamed from J4; footprint PinSocket_2x14_P2.54mm_Vertical -> MKR1010:PinSocket_2x14_MKR1010
- SW1: renamed from SW2; value StSp -> StSp - Farnell 986-501; footprint (none) -> MKR1010:jumper-switch
- SW2: renamed from SW3; value Sleep -> Sleep - Farnell 986-501; footprint (none) -> MKR1010:jumper-switch
- SW3: renamed from SW1; footprint (none) -> MKR1010:switch
- renumbered D4 to D2, D5 to D3, D2 to D4, D3 to D5, R2 to R1, R11 to R10, R12 to R11, R13 to R12, R14 to R13, R17 to R14, R18 to R15, R15 to R16, R16 to R17, R6 to R2, R7 to R6, R8 to R7, R9 to R8, R10 to R9
Connections:
- net +3V3: now also J4.3 (Pin_3), J4.6 (Pin_6)
- net GND: now also R2.1, J2.1 (Pin_1), J3.1 (Pin_1), J3.2 (Pin_2), J4.1 (Pin_1), J4.4 (Pin_4), J5.1 (Pin_1); no longer R2.2
- net at D1.2 (A), R8.1, SW3.3 (C): now also J5.2 (Pin_2)
- net at R9.1: now also J1.1 (Pin_1), J2.2 (Pin_2)
- net at J6.D0 (Pin_9), R3.2: now also J4.2 (Pin_2)
- net at J6.D3 (Pin_12), R1.2: now also J4.5 (Pin_5)
- net at SW3.2 (B): now also J1.2 (Pin_2)
- net at D1.1 (K): now also R2.2; no longer R2.1
- no-connect marks 13 -> 14
Other:
- note added: "07/11/2019"
- note added: "3.3V/2"
- note added: "8 + 6 pin stackable header"
- note added: "IHM(1/2)"
- note added: "IHM(2/2)"
- note added: "L'embase "shunt" permet l'insertion\nd'une résistance de faible valeur\nqui offre la possibilité de la mesure\ndu courant ibat."
- note added: "Mesures des tensions\n(4 X diviseur par 2)"
- note added: "Régis Leruste"
- note added: "Shield MKR wifi 1010"
- note added: "T1"
- note added: "T2"
- note added: "VBAT1/2"
- note added: "VBAT2/2"
- note added: "VUSB/2"
- note removed: "3.3V"
- note removed: "4 X diviseur par 2\nCalibration"
- note removed: "GND"
- note removed: "IHM"
- note removed: "Pupitre"
- note removed: "VUSB"
- moved on the sheet: D1, D2, D3, D4, D5, R14, R15, R16, R17, R2, R4, R5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

Commit message: 2ème maj du 07/10/2019
Other:
- note added: "https://github.com/AIREL46/SCAO/raw/master/kicad/e-p-wifi-shield/e-p-wifi.png"
Changed lines of the file:
@@
 Text Notes 7491 5600 0    50   ~ 10
 Régis Leruste
+Text Notes 4716 5686 0    50   ~ 10
+https://github.com/AIREL46/SCAO/raw/master/kicad/e-p-wifi-shield/e-p-wifi.png
 $EndSCHEMATC

Commit message: Ajout du logo A3C
Parts:
- J4: footprint Connector_PinHeader_1.00mm:PinHeader_1x06_P1.00mm_Vertical -> Connector_PinHeader_2.54mm:PinHeader_1x06_P2.54mm_Vertical
Changed lines of the file:
@@
 F 0 "J4" H 3013 2998 50  0000 C CNN
 F 1 "Température" H 2867 2655 50  0000 C CNN
-F 2 "Connector_PinHeader_1.00mm:PinHeader_1x06_P1.00mm_Vertical" H 2851 3050 50  0001 C CNN
+F 2 "Connector_PinHeader_2.54mm:PinHeader_1x06_P2.54mm_Vertical" H 2851 3050 50  0001 C CNN
 F 3 "~" H 2851 3050 50  0001 C CNN
 	1    2851 3050

Commit message: Maj du 20/11/2019
Parts:
- added C2, C3, C4, C5: 0.1mF, Capacitor_THT:C_Disc_D3.0mm_W1.6mm_P2.50mm, symbol Device:C
- added R18: 4.7k, Resistor_THT:R_Axial_DIN0207_L6.3mm_D2.5mm_P7.62mm_Horizontal, symbol Device:R
- added SW4: BP APEM - Farnell 108-2512, MKR1010:BP, symbol Switch:SW_Push
- R11: value 4.7k -> 47k
Connections:
- net +3V3: now also SW4.1
- net GND: now also R11.1, C2.2, C3.2, C4.2, C5.2, R18.2; no longer R11.2
- net at J6.A0 (Pin_2), R6.2: now also C5.1, R18.1; no longer R10.1
- net at J6.A1 (Pin_3), R7.2: now also R13.1, C4.1; no longer R11.1
- net at J6.A2 (Pin_4), R12.1, R8.2: now also C3.1
- net at J6.A3 (Pin_5), R9.2: now also R10.1, C2.1; no longer R13.1
- net at J6.A5 (Pin_7): now also R11.2, SW4.2
- no-connect marks 14 -> 13
Other:
- note added: "meross"
- moved on the sheet: R10, R6, R7, R8, R9

Commit message: Copie des fichiers kicad de Mikaël
Parts:
- J6: footprint MKR1010:PinSocket_2x14_MKR1010 -> e-p-wifi-v2:PinSocket_2x14_MKR1010
- SW1, SW2: footprint MKR1010:jumper-switch -> e-p-wifi-v2:jumper-switch
- SW3: footprint MKR1010:switch -> e-p-wifi-v2:switch
- SW4: footprint MKR1010:BP -> e-p-wifi-v2:BP
Changed lines of the file:
@@
 F 0 "SW3" H 3303 4189 50  0000 C CNN
 F 1 "Conrad 711771" H 3602 4087 50  0000 C CNN
-F 2 "MKR1010:switch" H 3350 4100 50  0001 C CNN
+F 2 "e-p-wifi-v2:switch" H 3350 4100 50  0001 C CNN
 F 3 "https://produktinfo.conrad.com/datenblaetter/700000-724999/711771-da-01-en-MINI_SCHIEBESCHALTER_450302014072.PDF" H 3350 4100 50  0001 C CNN
 	1    3350 4100
@@
 F 0 "SW1" H 3346 5095 50  0000 C CNN
 F 1 "StSp - Farnell 986-501" H 3484 5175 50  0000 C CNN
-F 2 "MKR1010:jumper-switch" H 3346 5362 50  0001 C CNN
+F 2 "e-p-wifi-v2:jumper-switch" H 3346 5362 50  0001 C CNN
 F 3 "http://www.farnell.com/datasheets/58539.pdf?_ga=2.27608380.140208918.1573048803-1966718086.1557591461&_gac=1.121467258.1573048803.Cj0KCQiA-4nuBRCnARIsAHwyuPqR51EVzwLC_rjGxuRlpl_aeelUyUlwni0GneFg4tO4wrwk64y3RFoaAuRiEALw_wcB" H 3346 5362 50  0001 C CNN
 	1    3346 5362
@@
 F 0 "SW2" H 3346 5545 50  0000 C CNN
 F 1 "Sleep - Farnell 986-501" H 3641 5639 50  0000 C CNN
-F 2 "MKR1010:jumper-switch" H 3346 5812 50  0001 C CNN
+F 2 "e-p-wifi-v2:jumper-switch" H 3346 5812 50  0001 C CNN
 F 3 "http://www.farnell.com/datasheets/58539.pdf?_ga=2.27608380.140208918.1573048803-1966718086.1557591461&_gac=1.121467258.1573048803.Cj0KCQiA-4nuBRCnARIsAHwyuPqR51EVzwLC_rjGxuRlpl_aeelUyUlwni0GneFg4tO4wrwk64y3RFoaAuRiEALw_wcB" H 3346 5812 50  0001 C CNN
 	1    3346 5812
@@
 F 0 "J6" V 6487 3697 100 0000 R CNB
 F 1 "Conn_02x14_MKR1010" V 6479 3339 75  0001 R CNB
-F 2 "MKR1010:PinSocket_2x14_MKR1010" V 6249 2680 50  0001 C CNN
+F 2 "e-p-wifi-v2:PinSocket_2x14_MKR1010" V 6249 2680 50  0001 C CNN
 F 3 "~" H 6100 2750 50  0001 C CNN
 	1    6100 2750
@@
 F 0 "SW4" H 3350 6300 50  0000 C CNN
 F 1 "BP APEM - Farnell 108-2512" H 3500 6600 50  0000 C CNN
-F 2 "MKR1010:BP" H 3350 6650 50  0001 C CNN
+F 2 "e-p-wifi-v2:BP" H 3350 6650 50  0001 C CNN
 F 3 "http://www.farnell.com/datasheets/10672.pdf?_ga=1.98306207.1823820493.1466675868" H 3350 6650 50  0001 C CNN
 	1    3350 6450
