File: kicad/e-p-wifi-shield/e-p-wifi.kicad_pcb (KiCad board)
At the start: 2 copper layers, 68.6 x 86.4 mm, 40 parts, among them J1 Shunt, J2 Vbat1, J3 Masse T1, J4 Température, J5 Vbat2, J6 Conn_02x14_MKR1010, SW1 StSp, SW2 Sleep, SW3 Conrad 711771, SW4 BP APEM

Commit message: mise à jour kicad
Parts:
- added C6: 0.1mF, Capacitor_THT:C_Disc_D3.0mm_W1.6mm_P2.50mm, F.Cu at (80.6, 104.1)
- added LH1: Via-DIY, e-p-wifi-v2:Via-DIY, F.Cu at (76.2, 80.0)
- added LH2: Via-DIY, e-p-wifi-v2:Via-DIY, F.Cu at (76.2, 57.1)
- added LH3: Via-DIY, e-p-wifi-v2:Via-DIY, F.Cu at (43.2, 68.6)
- added MH1: Via-DIY, e-p-wifi-v2:Via-DIY, F.Cu at (88.3, 58.4)
- added MH2: Via-DIY, e-p-wifi-v2:Via-DIY, F.Cu at (88.3, 78.7)
- added MH3: Via-DIY, e-p-wifi-v2:Via-DIY, F.Cu at (31.1, 58.4)
- added MH4: Via-DIY, e-p-wifi-v2:Via-DIY, F.Cu at (31.1, 78.7)
- J4: footprint Connector_PinHeader_2.54mm:PinHeader_1x06_P2.54mm_Vertical -> e-p-wifi-v2:PinHeader_1x06_P2.54mm_Vertical_J4
- J6: footprint e-p-wifi-v2:PinSocket_2x14_MKR1010 -> e-p-wifi-v2:PinSocket_2x14_MKR1010_ov
- SW1: value StSp -> StSp - Farnell 986-501; footprint e-p-wifi-v2:jumper-switch -> e-p-wifi-v2:jumper-switch-sw1
- SW2: value Sleep -> Sleep - Farnell 986-501; footprint e-p-wifi-v2:jumper-switch -> e-p-wifi-v2:jumper-switch-sw2
- SW4: value BP APEM -> BP APEM - Farnell 108-2512
- moved J4 30.5 mm to (22.9, 62.2), turned to 0 degrees
- moved J3 25.8 mm to (22.9, 79.4), turned to 0 degrees
- moved R4 2.20 mm to (42.5, 62.9)
Routing:
- net Net-(J4-Pad2): track 61.1 -> 35.1 mm
- net Net-(D5-Pad2): track 53.0 -> 31.0 mm
- net +3V3: track 137.9 -> 119.2 mm, vias 4 -> 0
- net Net-(J1-Pad2): track 107.6 -> 93.0 mm
- net Net-(J6-PadD2): track 90.9 -> 76.6 mm, vias 5 -> 0
- net Net-(J1-Pad1): track 80.0 -> 69.3 mm
- net Net-(D3-Pad2): track 85.6 -> 76.4 mm
- net Net-(J6-Pad+5V): track 25.3 -> 16.4 mm, vias 1 -> 0
- net Net-(J4-Pad5): track 55.0 -> 46.5 mm, vias 2 -> 0
- net Net-(J6-PadD1): track 81.3 -> 73.7 mm
- net Net-(C3-Pad1): track 47.6 -> 40.8 mm, vias 1 -> 0
- net Net-(D1-Pad2): track 145.6 -> 138.8 mm, vias 2 -> 0
- net Net-(C5-Pad1): track 46.5 -> 41.8 mm, vias 3 -> 0
- net Net-(C2-Pad1): track 59.7 -> 55.5 mm, vias 2 -> 0
- net Net-(D2-Pad2): track 67.9 -> 70.8 mm
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- added copper zone on B.Cu, net GND
Other:
- board size 68.6 x 86.4 mm -> 76.2 x 86.4 mm
