File: kicad/e-p-wifi-shield/e-p-wifi.kicad_pcb (KiCad board)
At the start: 2 copper layers, 76.2 x 86.4 mm, 48 parts, among them J1 Shunt, J2 Vbat1, J3 Masse T1, J4 Température, J5 Vbat2, J6 Conn_02x14_MKR1010, SW1 StSp - Farnell 986-501, SW2 Sleep - Farnell 986-501, SW3 Conrad 711771, SW4 BP APEM - Farnell 108-2512

Commit message: Mise à jour régis
Parts:
- removed C2: 0.1mF, Capacitor_THT:C_Disc_D3.0mm_W1.6mm_P2.50mm
- added J7: RJ45, Connector_RJ:RJ45_Wuerth_7499010001A_Horizontal, F.Cu at (1.51, 37.6)
- added LS1: Speaker, e-p-wifi:mini_speaker, F.Cu at (80.4, 30.4)
- added Q1: 2N2222A, Package_TO_SOT_THT:TO-18-3, F.Cu at (72.1, 39.6)
- added R9: 470, Resistor_THT:R_Axial_DIN0207_L6.3mm_D2.5mm_P7.62mm_Horizontal, F.Cu at (53.1, 33.7)
- J2: value Vbat1 -> Vbat
- J4: value Température -> T1; footprint e-p-wifi-v2:PinHeader_1x06_P2.54mm_Vertical_J4 -> Connector_PinHeader_2.54mm:PinHeader_1x03_P2.54mm_Vertical
- J5: value Vbat2 -> T2; footprint Connector_PinHeader_2.54mm:PinHeader_1x02_P2.54mm_Vertical -> Connector_PinHeader_2.54mm:PinHeader_1x03_P2.54mm_Vertical
- R10: value 4.7k -> 47k
- moved J5 74.9 mm to (22.7, 71.5), turned to 0 degrees
- moved J1 9.24 mm to (90.4, 40.6)
- moved R7 5.93 mm to (64.8, 94.0)
- moved R18 5.84 mm to (48.3, 86.4)
- moved C4 5.80 mm to (61.6, 86.4)
- moved R13 5.77 mm to (58.4, 86.4)
- moved C5 5.66 mm to (51.4, 86.4)
- moved R6 5.59 mm to (54.6, 94.0)
- moved R12 3.28 mm to (71.1, 86.4)
- moved C3 3.03 mm to (74.2, 86.4)
- moved R8 2.88 mm to (77.2, 94.0)
- moved J3 1.57 mm to (22.7, 80.9)
- moved R9 1.42 mm to (84.8, 93.2)
- moved J4 0.20 mm to (22.7, 62.4)
Connections:
- J5 pad 2: Net-(D1-Pad2) -> Net-(J5-Pad2)
- J6 pad A3: Net-(C2-Pad1) -> Net-(J6-PadA3)
- J6 pad A5: Net-(C6-Pad1) -> Net-(J6-PadA5)
- J6 pad D0: Net-(J4-Pad2) -> Net-(J5-Pad2)
- J6 pad D3: Net-(J4-Pad5) -> Net-(J4-Pad2)
- R1 pad 2: Net-(J4-Pad5) -> Net-(J4-Pad2)
- R10 pad 1: Net-(C2-Pad1) -> Net-(J6-PadA3)
- R11 pad 2: Net-(C6-Pad1) -> Net-(J6-PadA5)
- R3 pad 2: Net-(J4-Pad2) -> Net-(J5-Pad2)
- SW4 pad 2: Net-(C6-Pad1) -> Net-(J6-PadA5)
- SW4 pad 3: GND -> (no net)
- SW4 pad 4: GND -> (no net)
Routing:
- net GND: track 2.54 -> 114.9 mm
- net Net-(D1-Pad2): track 138.8 -> 63.3 mm
- net Net-(C2-Pad1): track 55.5 -> 0.00 mm
- net Net-(J6-PadA3): track 0.00 -> 54.2 mm
- net Net-(J4-Pad5): track 46.5 -> 0.00 mm
- net Net-(J5-Pad2): track 0.00 -> 44.3 mm
- net Net-(D2-Pad2): track 70.8 -> 83.5 mm
- net +3V3: track 119.2 -> 130.0 mm
- net Net-(C5-Pad1): track 41.8 -> 52.0 mm
- net Net-(J4-Pad2): track 35.1 -> 43.1 mm
- net Net-(D3-Pad2): track 76.4 -> 83.1 mm
- net Net-(C4-Pad1): track 42.0 -> 46.2 mm
- net Net-(J1-Pad1): track 69.3 -> 65.4 mm
- net Net-(J1-Pad2): track 93.0 -> 89.6 mm
- net Net-(J6-PadD2): track 76.6 -> 77.8 mm
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- removed copper zone on B.Cu, net GND
- removed copper zone on F.Cu, net GND
