File: kicad/e-r-wifi/e-r-wifi.sch (KiCad schematic (older format))
At the start: 7 parts, among them J1 Entrée 230V, J2 Sortie 230V, J3 cde relais Celduc, J4 5V, U1 SKL10120, U2 PC817

Commit message: Mise à jour
Parts:
- D1: footprint (none) -> Diode_THT:D_5KPW_P7.62mm_Vertical_AnodeUp
- J3, J4: footprint (none) -> Connector_PinHeader_2.54mm:PinHeader_1x02_P2.54mm_Horizontal
Changed lines of the file:
@@
 F 0 "J3" H 2600 2200 50  0000 C CNN
 F 1 "cde relais Celduc" H 2750 2100 50  0000 C CNN
-F 2 "" H 2600 2000 50  0001 C CNN
+F 2 "Connector_PinHeader_2.54mm:PinHeader_1x02_P2.54mm_Horizontal" H 2600 2000 50  0001 C CNN
 F 3 "~" H 2600 2000 50  0001 C CNN
 	1    2600 2000
@@
 F 0 "J4" H 2600 1550 50  0000 C CNN
 F 1 "5V" H 2600 1450 50  0000 C CNN
-F 2 "" H 2600 1350 50  0001 C CNN
+F 2 "Connector_PinHeader_2.54mm:PinHeader_1x02_P2.54mm_Horizontal" H 2600 1350 50  0001 C CNN
 F 3 "~" H 2600 1350 50  0001 C CNN
 	1    2600 1350
@@
 F 0 "D1" H 2943 2217 50  0000 C CNN
 F 1 "LED" H 2943 2126 50  0000 C CNN
-F 2 "" H 2950 2000 50  0001 C CNN
+F 2 "Diode_THT:D_5KPW_P7.62mm_Vertical_AnodeUp" H 2950 2000 50  0001 C CNN
 F 3 "https://asset.conrad.com/media10/add/160267/c1/-/en/000180129DS01/fiche-technique-180129-led-3-mm-jaune-kingbright-l-7104yd-l-7104yd-rond-15-mcd-40-20-ma-21-v-1-pcs.pdf" H 2950 2000 50  0001 C CNN
 	1    2950 2000

Commit message: mise à jour
Parts:
- D1: footprint Diode_THT:D_5KPW_P7.62mm_Vertical_AnodeUp -> Diode_THT:D_A-405_P2.54mm_Vertical_AnodeUp
- J3, J4: footprint Connector_PinHeader_2.54mm:PinHeader_1x02_P2.54mm_Horizontal -> Connector_PinHeader_2.54mm:PinHeader_1x02_P2.54mm_Vertical
- U1: symbol Relay_SolidState:FODM3053 -> Relay_SolidState:S102S01
Changed lines of the file:
@@
 $EndComp
 $Comp
-L Relay_SolidState:FODM3053 U1
+L Relay_SolidState:S102S01 U1
 U 1 1 5FACEE00
 P 4000 1900
@@
 F 0 "J3" H 2600 2200 50  0000 C CNN
 F 1 "cde relais Celduc" H 2750 2100 50  0000 C CNN
-F 2 "Connector_PinHeader_2.54mm:PinHeader_1x02_P2.54mm_Horizontal" H 2600 2000 50  0001 C CNN
+F 2 "Connector_PinHeader_2.54mm:PinHeader_1x02_P2.54mm_Vertical" H 2600 2000 50  0001 C CNN
 F 3 "~" H 2600 2000 50  0001 C CNN
 	1    2600 2000
@@
 F 0 "J4" H 2600 1550 50  0000 C CNN
 F 1 "5V" H 2600 1450 50  0000 C CNN
-F 2 "Connector_PinHeader_2.54mm:PinHeader_1x02_P2.54mm_Horizontal" H 2600 1350 50  0001 C CNN
+F 2 "Connector_PinHeader_2.54mm:PinHeader_1x02_P2.54mm_Vertical" H 2600 1350 50  0001 C CNN
 F 3 "~" H 2600 1350 50  0001 C CNN
 	1    2600 1350
@@
 F 0 "D1" H 2943 2217 50  0000 C CNN
 F 1 "LED" H 2943 2126 50  0000 C CNN
-F 2 "Diode_THT:D_5KPW_P7.62mm_Vertical_AnodeUp" H 2950 2000 50  0001 C CNN
+F 2 "Diode_THT:D_A-405_P2.54mm_Vertical_AnodeUp" H 2950 2000 50  0001 C CNN
 F 3 "https://asset.conrad.com/media10/add/160267/c1/-/en/000180129DS01/fiche-technique-180129-led-3-mm-jaune-kingbright-l-7104yd-l-7104yd-rond-15-mcd-40-20-ma-21-v-1-pcs.pdf" H 2950 2000 50  0001 C CNN
 	1    2950 2000

Commit message: mise à jour
Parts:
- D1: value LED -> LED
Changed lines of the file:
@@
 P 2950 2000
 F 0 "D1" H 2943 2217 50  0000 C CNN
-F 1 "LED" H 2943 2126 50  0000 C CNN
+F 1 "LED " H 2943 2126 50  0000 C CNN
 F 2 "Diode_THT:D_A-405_P2.54mm_Vertical_AnodeUp" H 2950 2000 50  0001 C CNN
 F 3 "https://asset.conrad.com/media10/add/160267/c1/-/en/000180129DS01/fiche-technique-180129-led-3-mm-jaune-kingbright-l-7104yd-l-7104yd-rond-15-mcd-40-20-ma-21-v-1-pcs.pdf" H 2950 2000 50  0001 C CNN
