File: kicad/e-r-wifi/e-r-wifi.kicad_pcb (KiCad board)
At the start: 2 copper layers, 7 parts, among them J1 Entrée 230V, J2 Sortie 230V, J3 cde relais Celduc, J4 5V, U1 SKL10120, U2 PC817

Commit message: mise à jour
Parts:
- D1: footprint Diode_THT:D_5KPW_P7.62mm_Vertical_AnodeUp -> Diode_THT:D_A-405_P2.54mm_Vertical_AnodeUp
- J3, J4: footprint Connector_PinHeader_2.54mm:PinHeader_1x02_P2.54mm_Horizontal -> Connector_PinHeader_2.54mm:PinHeader_1x02_P2.54mm_Vertical
- moved J2 75.1 mm to (154.9, 49.5), turned to 90 degrees
- moved J1 45.4 mm to (105.4, 49.5), turned to 90 degrees
- moved J3 45.3 mm to (105.4, 57.1)
- moved J4 30.6 mm to (105.4, 66.0)
- moved U2 26.1 mm to (113.0, 62.2), turned to 270 degrees
- moved U1 24.8 mm to (142.2, 58.1), turned to 180 degrees
- moved D1 14.4 mm to (113.0, 57.1), turned to 180 degrees
Connections:
- U1 pad 1: Net-(J4-Pad1) -> Net-(J2-Pad1)
- U1 pad 2: Net-(U1-Pad2) -> Net-(J1-Pad1)
- U1 pad 3: Net-(J1-Pad1) -> Net-(J4-Pad1)
- U1 pad 4: Net-(J2-Pad1) -> Net-(U1-Pad4)
- U2 pad 4: Net-(U1-Pad2) -> Net-(U1-Pad4)
Routing:
- net Net-(J4-Pad1): track 0.00 -> 71.2 mm
- net Net-(J1-Pad3): track 0.00 -> 49.5 mm
- net Net-(J1-Pad2): track 0.00 -> 49.5 mm
- net Net-(U1-Pad4): track 0.00 -> 44.8 mm
- net Net-(J1-Pad1): track 0.00 -> 28.8 mm
- net Net-(J2-Pad1): track 0.00 -> 27.5 mm
- net Net-(D1-Pad2): track 0.00 -> 8.89 mm
- net Net-(J3-Pad2): track 0.00 -> 7.54 mm
- net GND: track 0.00 -> 6.35 mm
- net Net-(D1-Pad1): track 0.00 -> 5.08 mm
Other:
- board outline added: 63.8 x 45.9 mm

Commit message: Mise à jour
Parts:
- moved U1 13.1 mm to (137.3, 70.3), turned to 0 degrees
Routing:
- net Net-(U1-Pad4): track 44.8 -> 13.0 mm
- net Net-(J4-Pad1): track 71.2 -> 43.4 mm
- net Net-(J1-Pad1): track 28.8 -> 47.4 mm
- net Net-(J2-Pad1): track 27.5 -> 21.2 mm
Other:
- board size 63.8 x 45.9 mm -> 63 x 50.4 mm

Commit message: mise à jour
Routing:
- net Net-(J1-Pad1): track 47.4 -> 46.8 mm

Commit message: mise à jour
Parts:
- D1: value LED -> LED
Changed lines of the file:
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@@
-      (effects (font (size 1 1) (thickness 0.15)))
-    )
-    (fp_text user %R (at 5.08 -0.5 90) (layer F.Fab)
       (effects (font (size 1 1) (thickness 0.15)))
     )
@@
     (fp_line (start 0.8 -1.2) (end 0 0) (layer F.Fab) (width 0.1))
     (fp_line (start 0 0) (end -0.8 -1.2) (layer F.Fab) (width 0.1))
+    (fp_text user %R (at 5.08 -0.5 90) (layer F.Fab)
+      (effects (font (size 1 1) (thickness 0.15)))
+    )
     (pad 3 thru_hole oval (at 10.16 0 90) (size 1.8 3.6) (drill 1.2) (layers *.Cu *.Mask)
       (net 5 "Net-(J1-Pad3)"))
@@
     )
     (fp_text value "Sortie 230V" (at 5.08 9.2 90) (layer F.Fab)
-      (effects (font (size 1 1) (thickness 0.15)))
-    )
-    (fp_text user %R (at 5.08 -0.5 90) (layer F.Fab)
       (effects (font (size 1 1) (thickness 0.15)))
     )
@@
     (fp_line (start 0.8 -1.2) (end 0 0) (layer F.Fab) (width 0.1))
     (fp_line (start 0 0) (end -0.8 -1.2) (layer F.Fab) (width 0.1))
+    (fp_text user %R (at 5.08 -0.5 90) (layer F.Fab)
+      (effects (font (size 1 1) (thickness 0.15)))
+    )
     (pad 3 thru_hole oval (at 10.16 0 90) (size 1.8 3.6) (drill 1.2) (layers *.Cu *.Mask)
       (net 5 "Net-(J1-Pad3)"))
@@
       (effects (font (size 1 1) (thickness 0.15)))
     )
-    (fp_text user %R (at 1.27 1.27 90) (layer F.Fab)
-      (effects (font (size 1 1) (thickness 0.15)))
-    )
-    (fp_arc (start 3.81 -1.33) (end 2.81 -1.33) (angle -180) (layer F.SilkS) (width 0.12))
     (fp_line (start 1.635 -1.27) (end 6.985 -1.27) (layer F.Fab) (width 0.1))
     (fp_line (start 6.985 -1.27) (end 6.985 3.81) (layer F.Fab) (width 0.1))
@@
     (fp_line (start 8.7 4.1) (end 8.7 -1.55) (layer F.CrtYd) (width 0.05))
     (fp_line (start 8.7 -1.55) (end -1.1 -1.55) (layer F.CrtYd) (width 0.05))
+    (fp_text user %R (at 1.27 1.27 90) (layer F.Fab)
+      (effects (font (size 1 1) (thickness 0.15)))
+    )
+    (fp_arc (start 3.81 -1.33) (end 2.81 -1.33) (angle -180) (layer F.SilkS) (width 0.12))
     (pad 4 thru_hole oval (at 7.62 0 270) (size 1.6 1.6) (drill 0.8) (layers *.Cu *.Mask)
       (net 10 "Net-(U1-Pad4)"))
@@
       (effects (font (size 1 1) (thickness 0.15)))
     )
-    (fp_text value LED (at 1.27 3.359) (layer F.Fab)
-      (effects (font (size 1 1) (thickness 0.15)))
-    )
-    (fp_text user A (at 4.44 0) (layer F.SilkS)
-      (effects (font (size 1 1) (thickness 0.15)))
-    )
-    (fp_text user A (at 4.44 0) (layer F.Fab)
-      (effects (font (size 1 1) (thickness 0.15)))
-    )
-    (fp_text user %R (at 1.27 -2.47) (layer F.Fab)
-      (effects (font (size 1 1) (thickness 0.15)))
-    )
-    (fp_arc (start 0 0) (end 1.113239 -0.9) (angle -278.451986) (layer F.SilkS) (width 0.12))
+    (fp_text value "LED " (at 1.27 3.359) (layer F.Fab)
+      (effects (font (size 1 1) (thickness 0.15)))
+    )
     (fp_circle (center 0 0) (end 1.35 0) (layer F.Fab) (width 0.1))
     (fp_line (start 0 0) (end 2.54 0) (layer F.Fab) (width 0.1))
@@
     (fp_line (start 3.69 1.6) (end 3.69 -1.6) (layer F.CrtYd) (width 0.05))
     (fp_line (start 3.69 -1.6) (end -1.6 -1.6) (layer F.CrtYd) (width 0.05))
+    (fp_text user A (at 4.44 0) (layer F.SilkS)
+      (effects (font (size 1 1) (thickness 0.15)))
+    )
+    (fp_text user A (at 4.44 0) (layer F.Fab)
+      (effects (font (size 1 1) (thickness 0.15)))
+    )
+    (fp_text user %R (at 1.27 -2.47) (layer F.Fab)
+      (effects (font (size 1 1) (thickness 0.15)))
+    )
+    (fp_arc (start 0 0) (end 1.113239 -0.9) (angle -278.451986) (layer F.SilkS) (width 0.12))
     (pad 2 thru_hole oval (at 2.54 0 180) (size 1.8 1.8) (drill 0.9) (layers *.Cu *.Mask)
       (net 2 "Net-(D1-Pad2)"))
@@
     )
     (fp_text value "cde relais Celduc" (at 0 4.87) (layer F.Fab)
-      (effects (font (size 1 1) (thickness 0.15)))
-    )
-    (fp_text user %R (at 0 1.27 90) (layer F.Fab)
       (effects (font (size 1 1) (thickness 0.15)))
     )
@@
     (fp_line (start 1.8 4.35) (end 1.8 -1.8) (layer F.CrtYd) (width 0.05))
     (fp_line (start 1.8 -1.8) (end -1.8 -1.8) (layer F.CrtYd) (width 0.05))
+    (fp_text user %R (at 0 1.27 90) (layer F.Fab)
+      (effects (font (size 1 1) (thickness 0.15)))
+    )
     (pad 2 thru_hole oval (at 0 2.54) (size 1.7 1.7) (drill 1) (layers *.Cu *.Mask)
       (net 7 "Net-(J3-Pad2)"))
@@
     )
     (fp_text value 5V (at 0 4.87) (layer F.Fab)
-      (effects (font (size 1 1) (thickness 0.15)))
-    )
-    (fp_text user %R (at 0 1.27 90) (layer F.Fab)
       (effects (font (size 1 1) (thickness 0.15)))
     )
@@
     (fp_line (start 1.8 4.35) (end 1.8 -1.8) (layer F.CrtYd) (width 0.05))
     (fp_line (start 1.8 -1.8) (end -1.8 -1.8) (layer F.CrtYd) (width 0.05))
+    (fp_text user %R (at 0 1.27 90) (layer F.Fab)
+      (effects (font (size 1 1) (thickness 0.15)))
+    )
     (pad 2 thru_hole oval (at 0 2.54) (size 1.7 1.7) (drill 1) (layers *.Cu *.Mask)
       (net 8 GND))

Commit message: mise à jour
Parts:
- moved J2 1.29 mm to (153.7, 49.5)
- moved U1 0.43 mm to (137.3, 69.9)
Connections:
- J3 pad 2: Net-(J3-Pad2) -> Net-(D1-Pad2)
- U2 pad 2: Net-(J3-Pad2) -> Net-(D1-Pad2)
Routing:
- net Net-(J4-Pad1): track 43.4 -> 29.1 mm
- net Net-(J3-Pad2): track 7.54 -> 0.00 mm
- net Net-(D1-Pad2): track 8.89 -> 16.4 mm
- net Net-(U1-Pad4): track 13.0 -> 15.3 mm
- net Net-(J1-Pad1): track 46.8 -> 48.1 mm
- net Net-(J2-Pad1): track 21.2 -> 22.1 mm
- net GND: track 6.35 -> 5.61 mm

Commit message: mise à jour
Parts:
- moved J2 37.2 mm to (160.9, 86.0)
- moved U1 37.2 mm to (144.6, 106.3)
- moved D1 37.2 mm to (120.3, 93.6)
- moved J3 37.2 mm to (112.7, 93.6)
- moved U2 37.2 mm to (120.3, 98.7)
- moved J1 37.2 mm to (112.7, 86.0)
- moved J4 37.2 mm to (112.7, 102.5)
Routing:
- net Net-(J1-Pad1): track 48.1 -> 46.7 mm
- added copper zone on B.Cu, net (none)
Other:
- board size 63 x 50.4 mm -> 66 x 59 mm
