File: kicad/e-r-wifi/e-r-wifi.kicad_pcb (KiCad board)
At the start: 2 copper layers, 66 x 59 mm, 7 parts, among them J1 Entrée 230V, J2 Sortie 230V, J3 cde relais Celduc, J4 5V, U1 SKL10120, U2 PC817

Commit message: mise à jour
Other:
- board size 66 x 59 mm -> 73 x 59 mm
- board text added: "CC-BY 28/05/2021 Olivier Marais"
- board text added: "e-rupteur e-r-wifi"
- board text added: "https://github.com/AIREL46/SCAO/blob/"
- board text added: "master/kicad/e-r-wifi/e-r-wifi.kicad_pcb"
