File: kicad/e-p-wifi/e-p-wifi.sch (KiCad schematic (older format))
At the start: 32 parts, among them J2 T1, J3 Masse, J4 T2, SW1 ON/OFF, SW2 StSp, SW3 Sleep, U1 Arduino_MKR_WIFI_1010

Commit message: Copie des fichiers kicad de Mikaël
Parts:
- removed BT1: Battery_Cell, symbol Device:Battery_Cell
- removed J2: T1, symbol Connector:Conn_01x03_Male
- removed J3: Masse, symbol Connector:Conn_01x01_Male
- removed J4: T2, symbol Connector:Conn_01x03_Male
- removed R1: 1 Ohm, symbol Device:R
- removed R10, R14: 4.7k, symbol Device:R
- removed U1: Arduino_MKR_WIFI_1010, symbol e-p-wifi-rescue:Arduino_MKR_WIFI_1010-MCU_Module
- added C2, C3, C4, C5: 0.1mF, Capacitor_THT:C_Disc_D3.0mm_W1.6mm_P2.50mm, symbol Device:C
- added J1: Shunt, Connector_PinHeader_2.54mm:PinHeader_1x02_P2.54mm_Vertical, symbol Connector_Generic:Conn_01x02
- added J2: Vbat1, Connector_PinHeader_2.54mm:PinHeader_1x02_P2.54mm_Vertical, symbol Connector_Generic:Conn_01x02
- added J3: Masse T1, Connector_PinHeader_2.54mm:PinHeader_1x02_P2.54mm_Vertical, symbol Connector_Generic:Conn_01x02
- added J4: Température, Connector_PinHeader_2.54mm:PinHeader_1x06_P2.54mm_Vertical, symbol Connector_Generic:Conn_01x06
- added J5: Vbat2, Connector_PinHeader_2.54mm:PinHeader_1x02_P2.54mm_Vertical, symbol Connector_Generic:Conn_01x02
- added J6: Conn_02x14_MKR1010, e-p-wifi-v2:PinSocket_2x14_MKR1010, symbol e-p-wifi-rescue:Conn_02x14_MKR1010
- added R11: 47k, Resistor_THT:R_Axial_DIN0207_L6.3mm_D2.5mm_P7.62mm_Horizontal, symbol Device:R
- added R13, R18: 4.7k, Resistor_THT:R_Axial_DIN0207_L6.3mm_D2.5mm_P7.62mm_Horizontal, symbol Device:R
- added SW4: BP APEM - Farnell 108-2512, e-p-wifi-v2:BP, symbol Switch:SW_Push
- C1: footprint (none) -> Capacitor_THT:CP_Radial_D5.0mm_P2.50mm
- D1: footprint (none) -> LED_THT:LED_D3.0mm
- D2: renamed from D5; footprint (none) -> LED_THT:LED_D3.0mm
- D3: renamed from D2; footprint (none) -> LED_THT:LED_D3.0mm
- D4: renamed from D3; footprint (none) -> LED_THT:LED_D3.0mm
- D5: renamed from D4; footprint (none) -> LED_THT:LED_D3.0mm
- R1: renamed from R4; footprint (none) -> Resistor_THT:R_Axial_DIN0207_L6.3mm_D2.5mm_P7.62mm_Horizontal
- R10: renamed from R8; footprint (none) -> Resistor_THT:R_Axial_DIN0207_L6.3mm_D2.5mm_P7.62mm_Horizontal
- R12, R15, R16, R17: footprint (none) -> Resistor_THT:R_Axial_DIN0207_L6.3mm_D2.5mm_P7.62mm_Horizontal
- R14: renamed from R18; footprint (none) -> Resistor_THT:R_Axial_DIN0207_L6.3mm_D2.5mm_P7.62mm_Horizontal
- R2: renamed from R1; footprint (none) -> Resistor_THT:R_Axial_DIN0207_L6.3mm_D2.5mm_P7.62mm_Horizontal
- R3: renamed from R5; footprint (none) -> Resistor_THT:R_Axial_DIN0207_L6.3mm_D2.5mm_P7.62mm_Horizontal
- R4: renamed from R2; footprint (none) -> Resistor_THT:R_Axial_DIN0207_L6.3mm_D2.5mm_P7.62mm_Horizontal
- R5: renamed from R3; footprint (none) -> Resistor_THT:R_Axial_DIN0207_L6.3mm_D2.5mm_P7.62mm_Horizontal
- R6: renamed from R7; footprint (none) -> Resistor_THT:R_Axial_DIN0207_L6.3mm_D2.5mm_P7.62mm_Horizontal
- R7: renamed from R9; footprint (none) -> Resistor_THT:R_Axial_DIN0207_L6.3mm_D2.5mm_P7.62mm_Horizontal
- R8: renamed from R11; footprint (none) -> Resistor_THT:R_Axial_DIN0207_L6.3mm_D2.5mm_P7.62mm_Horizontal
- R9: renamed from R13; footprint (none) -> Resistor_THT:R_Axial_DIN0207_L6.3mm_D2.5mm_P7.62mm_Horizontal
- SW1: renamed from SW2; value StSp -> StSp - Farnell 986-501; footprint (none) -> e-p-wifi-v2:jumper-switch
- SW2: renamed from SW3; value Sleep -> Sleep - Farnell 986-501; footprint (none) -> e-p-wifi-v2:jumper-switch
- SW3: renamed from SW1; value ON/OFF -> Conrad 711771; footprint (none) -> e-p-wifi-v2:switch
Connections:
- wire segments 120 -> 139
- no-connect marks 14 -> 13
Other:
- note added: "07/11/2019"
- note added: "3.3V/2"
- note added: "8 + 6 pin stackable header"
- note added: "IHM(1/2)"
- note added: "IHM(2/2)"
- note added: "L'embase "shunt" permet l'insertion\nd'une résistance de faible valeur\nqui offre la possibilité de la mesure\ndu courant ibat."
- note added: "Mesures des tensions\n(4 X diviseur par 2)"
- note added: "Régis Leruste"
- note added: "Shield MKR wifi 1010"
- note added: "T1"
- note added: "T2"
- note added: "VBAT1/2"
- note added: "VBAT2/2"
- note added: "VUSB/2"
- note added: "https://github.com/AIREL46/SCAO/raw/master/kicad/e-p-wifi-shield/e-p-wifi.png"
- note added: "meross"
- note removed: "+"
- note removed: "-"
- note removed: "3.3V"
- note removed: "4 X diviseur par 2\nCalibration"
- note removed: "Breadboard [3b]"
- note removed: "DS18B20"
- note removed: "Entretoise de fixation [16]"
- note removed: "GND"
- note removed: "IHM"
- note removed: "Pupitre"
- note removed: "VUSB"
- note removed: "[17]"
- note removed: "[4]"
- note removed: "[7]"
- moved on the sheet: D1, D2, D3, D4, D5, R10, R14, R15, R16, R17, R2, R4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

Commit message: Mise à jour Olivier
Parts:
- added J?: RJ45, Connector_RJ:RJ45_OST_PJ012-8P8CX_Vertical, symbol Connector:RJ45
- added LS?: Speaker, symbol Device:Speaker
- added Q?: 2N2219, Package_TO_SOT_THT:TO-39-3, symbol Transistor_BJT:2N2219
- added R?: R, symbol Device:R
Changed lines of the file:
@@
 EESchema Schematic File Version 4
-LIBS:e-p-wifi-cache
 EELAYER 30 0
 EELAYER END
@@
 Wire Notes Line
 	2848 1514 8220 1514
-Wire Notes Line
-	8220 1514 8220 6346
 Wire Notes Line
 	2848 6346 2848 2252
@@
 Wire Notes Line
 	2850 7150 2850 6350
+$Comp
+L Connector:RJ45 J?
+U 1 1 612B81E4
+P 8650 3250
+F 0 "J?" H 8320 3254 50  0000 R CNN
+F 1 "RJ45" H 8320 3345 50  0000 R CNN
+F 2 "Connector_RJ:RJ45_OST_PJ012-8P8CX_Vertical" V 8650 3275 50  0001 C CNN
+F 3 "~" V 8650 3275 50  0001 C CNN
+	1    8650 3250
+	-1   0    0    1
+$EndComp
+$Comp
+L Transistor_BJT:2N2219 Q?
+U 1 1 612CC513
+P 8700 2200
+F 0 "Q?" H 8890 2246 50  0000 L CNN
+F 1 "2N2219" H 8890 2155 50  0000 L CNN
+F 2 "Package_TO_SOT_THT:TO-39-3" H 8900 2125 50  0001 L CIN
+F 3 "http://www.onsemi.com/pub_link/Collateral/2N2219-D.PDF" H 8700 2200 50  0001 L CNN
+	1    8700 2200
+	1    0    0    -1
+$EndComp
+$Comp
+L Device:Speaker LS?
+U 1 1 612CE3C8
+P 8750 1650
+F 0 "LS?" H 8920 1646 50  0000 L CNN
+F 1 "Speaker" H 8920 1555 50  0000 L CNN
+F 2 "" H 8750 1450 50  0001 C CNN
+F 3 "~" H 8740 1600 50  0001 C CNN
+	1    8750 1650
+	1    0    0    -1
+$EndComp
+$Comp
+L Device:R R?
+U 1 1 612CF765
+P 8700 2600
+F 0 "R?" V 8493 2600 50  0000 C CNN
+F 1 "R" V 8584 2600 50  0000 C CNN
+F 2 "" V 8630 2600 50  0001 C CNN
+F 3 "~" H 8700 2600 50  0001 C CNN
+	1    8700 2600
+	0    1    1    0
+$EndComp
 $EndSCHEMATC

Commit message: Mise à jour Régis
Parts:
- removed R?: R, symbol Device:R
- added R?: 470, Resistor_THT:R_Axial_DIN0207_L6.3mm_D2.5mm_P7.62mm_Horizontal, symbol Device:R
- LS?: footprint (none) -> e-p-wifi:mini_speaker
- Q?: value 2N2219 -> 2N2222A; footprint Package_TO_SOT_THT:TO-39-3 -> Package_TO_SOT_THT:TO-18-3
Connections:
- net +3V3: now also Q?.3 (C)
- net GND: now also LS?.2
- net at J6.D4 (Pin_13): now also R?.2
- net at Q?.1 (E): now also LS?.1
- net at Q?.2 (B): now also R?.1
- no-connect marks 13 -> 12
Other:
- moved on the sheet: J?, LS?, Q?
Changed lines of the file:
@@
 NoConn ~ 5600 1750
 Wire Wire Line
-	5700 1750 5700 1670
-Wire Wire Line
 	5500 1750 5500 1700
-NoConn ~ 6700 2950
 Wire Wire Line
 	6000 2950 6000 3000
@@
 L Connector:RJ45 J?
 U 1 1 612B81E4
-P 8650 3250
-F 0 "J?" H 8320 3254 50  0000 R CNN
-F 1 "RJ45" H 8320 3345 50  0000 R CNN
-F 2 "Connector_RJ:RJ45_OST_PJ012-8P8CX_Vertical" V 8650 3275 50  0001 C CNN
-F 3 "~" V 8650 3275 50  0001 C CNN
-	1    8650 3250
+P 9800 1950
+F 0 "J?" H 9470 1954 50  0000 R CNN
+F 1 "RJ45" H 9470 2045 50  0000 R CNN
+F 2 "Connector_RJ:RJ45_OST_PJ012-8P8CX_Vertical" V 9800 1975 50  0001 C CNN
+F 3 "~" V 9800 1975 50  0001 C CNN
+	1    9800 1950
 	-1   0    0    1
 $EndComp
@@
 L Transistor_BJT:2N2219 Q?
 U 1 1 612CC513
-P 8700 2200
-F 0 "Q?" H 8890 2246 50  0000 L CNN
-F 1 "2N2219" H 8890 2155 50  0000 L CNN
-F 2 "Package_TO_SOT_THT:TO-39-3" H 8900 2125 50  0001 L CIN
-F 3 "http://www.onsemi.com/pub_link/Collateral/2N2219-D.PDF" H 8700 2200 50  0001 L CNN
-	1    8700 2200
+P 8500 3050
+F 0 "Q?" H 8690 3096 50  0000 L CNN
+F 1 "2N2222A" H 8690 3005 50  0000 L CNN
+F 2 "Package_TO_SOT_THT:TO-18-3" H 8700 2975 50  0001 L CIN
+F 3 "http://www.onsemi.com/pub_link/Collateral/2N2219-D.PDF" H 8500 3050 50  0001 L CNN
+	1    8500 3050
 	1    0    0    -1
 $EndComp
@@
 L Device:Speaker LS?
 U 1 1 612CE3C8
-P 8750 1650
-F 0 "LS?" H 8920 1646 50  0000 L CNN
-F 1 "Speaker" H 8920 1555 50  0000 L CNN
-F 2 "" H 8750 1450 50  0001 C CNN
-F 3 "~" H 8740 1600 50  0001 C CNN
-	1    8750 1650
-	1    0    0    -1
-$EndComp
+P 8800 3500
+F 0 "LS?" H 8970 3496 50  0000 L CNN
+F 1 "Speaker" H 8970 3405 50  0000 L CNN
+F 2 "e-p-wifi:mini_speaker" H 8800 3300 50  0000 C CNN
+F 3 "http://cdn.sparkfun.com/datasheets/Components/General/cem-1203-42-.pdf" H 8790 3450 50  0001 C CNN
+	1    8800 3500
+	1    0    0    -1
+$EndComp
+Wire Wire Line
+	8000 3050 6700 3050
+Wire Wire Line
+	6700 3050 6700 2950
+Wire Wire Line
+	8600 3250 8600 3500
+$Comp
+L power:GND #PWR?
+U 1 1 615137D3
+P 8600 3750
+F 0 "#PWR?" H 8600 3500 50  0001 C CNN
+F 1 "GND" H 8605 3577 50  0000 C CNN
+F 2 "" H 8600 3750 50  0001 C CNN
+F 3 "" H 8600 3750 50  0001 C CNN
+	1    8600 3750
+	1    0    0    -1
+$EndComp
+Wire Wire Line
+	8600 3750 8600 3600
+Wire Wire Line
+	8600 2850 8600 1550
+Wire Wire Line
+	8600 1550 5700 1550
+Wire Wire Line
+	5700 1550 5700 1670
+Connection ~ 5700 1670
+Wire Wire Line
+	5700 1670 5700 1750
 $Comp
 L Device:R R?
-U 1 1 612CF765
-P 8700 2600
-F 0 "R?" V 8493 2600 50  0000 C CNN
-F 1 "R" V 8584 2600 50  0000 C CNN
-F 2 "" V 8630 2600 50  0001 C CNN
-F 3 "~" H 8700 2600 50  0001 C CNN
-	1    8700 2600
+U 1 1 6152EC58
+P 8150 3050
+F 0 "R?" V 8149 2978 50  0000 L CNN
+F 1 "470" V 8050 3000 50  0000 L CNN
+F 2 "Resistor_THT:R_Axial_DIN0207_L6.3mm_D2.5mm_P7.62mm_Horizontal" V 8080 3050 50  0001 C CNN
+F 3 "~" H 8150 3050 50  0001 C CNN
+	1    8150 3050
 	0    1    1    0
 $EndComp

Commit message: Mise à jour Régis
Parts:
- removed C2: 0.1mF, Capacitor_THT:C_Disc_D3.0mm_W1.6mm_P2.50mm, symbol Device:C
- removed J4: Température, Connector_PinHeader_2.54mm:PinHeader_1x06_P2.54mm_Vertical, symbol Connector_Generic:Conn_01x06
- removed J5: Vbat2, Connector_PinHeader_2.54mm:PinHeader_1x02_P2.54mm_Vertical, symbol Connector_Generic:Conn_01x02
- removed R9: 4.7k, Resistor_THT:R_Axial_DIN0207_L6.3mm_D2.5mm_P7.62mm_Horizontal, symbol Device:R
- added J4: T1, symbol Connector_Generic:Conn_01x03
- added J5: T2, symbol Connector_Generic:Conn_01x03
- J2: value Vbat1 -> Vbat
- J7: renamed from J?; footprint Connector_RJ:RJ45_OST_PJ012-8P8CX_Vertical -> Connector_RJ:RJ45_Wuerth_7499010001A_Horizontal
- R10: value 4.7k -> 47k
- gave numbers to parts that had none: 3
Connections:
- net +3V3: now also J7.2, Q1.1 (E), J4.3 (Pin_3), J5.3 (Pin_3); no longer Q1.3 (C)
- net GND: now also J7.6, J7.7, J7.8, J4.1 (Pin_1), J5.1 (Pin_1)
- net at J6.A3 (Pin_5), R10.1: now also J7.5
- net at J6.+5V (Pin_28), R7.1: now also J7.1
- net at J6.D0 (Pin_9), R3.2: now also J5.2 (Pin_2)
- net at J6.D3 (Pin_12), R1.2: now also J4.2 (Pin_2)
- net at J6.A5 (Pin_7), R11.2, SW4.2: now also J7.4
- net at J6.A6 (Pin_8): now also J7.3
- net at LS1.1: now also Q1.3 (C); no longer Q1.1 (E)
- no-connect marks 12 -> 11
Other:
- note added: "+5V"
- note added: "Cde relais"
- note added: "Mesures des tensions\n(3 X diviseur par 2)"
- note added: "P230V"
- note added: "Pour le routage du transistor voir : \nhttps://fablabo.net/wiki/Atelier_logiciel#Routage_d.27un_transistor_sous_kicad"
- note added: "VBAT"
- note added: "VBAT/2"
- note added: "VCC"
- note added: "itc"
- note removed: "Mesures des tensions\n(4 X diviseur par 2)"
- note removed: "T1"
- note removed: "T2"
- note removed: "VBAT1"
- note removed: "VBAT1/2"
- note removed: "VBAT2"
- note removed: "VBAT2/2"
- note removed: "VDD"
- moved on the sheet: LS1, Q1, R9
