File: kicad/e-p-wifi-lf/e-p-wifi-lf.kicad_pcb (KiCad board)
At the start: 2 copper layers, 54.6 x 25.4 mm, 7 parts, among them J1 Speaker, J2 liaison_filaire, J3 RJ45, Q1 2N2222A

Commit message: Mise à jour Régis
Other:
- board text added: "e-p-wifi-lf"
Changed lines of the file:
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@@
   (general
     (thickness 1.6)
-    (drawings 23)
+    (drawings 24)
     (tracks 72)
     (zones 0)
@@
       (viasonmask false)
       (mode 1)
-      (useauxorigin false)
+      (useauxorigin true)
       (hpglpennumber 1)
       (hpglpenspeed 20)
@@
     )
   )
+  (gr_text e-p-wifi-lf (at 71.628 121.412) (layer B.Fab)
+    (effects (font (size 1 1) (thickness 0.15)) (justify mirror))
+  )
   (gr_line (start 95.25 134.62) (end 88.9 134.62) (layer Edge.Cuts) (width 0.05))
