File: kicad/e-p-wifi-lf/e-p-wifi-lf.sch (KiCad schematic (older format))
At the start: 7 parts, among them J1 Speaker, J2 liaison_filaire, J3 RJ45, Q1 2N2222A

Commit message: Mise à jour Régis
Parts:
- J2: value liaison_filaire -> 2 X Arduino Stackable Header - 8 Pin - Sparkfun PRT-09279; footprint e-p-wifi-lf:PinHeader_1x08 -> e-p-wifi-lf:PinHeader_2x08
- J3: value RJ45 -> RJ45-e-p-wifi-cache-e-p-wifi-lf-rescue; footprint e-p-wifi-lf:RJ45 -> (none)
- LS1: value Device_Speaker -> Mini speaker Sparkfun 07950
- Q1: value 2N2222A -> 2N2222A Conrad 1359807
Other:
- note added: "Source : https://fr.wikipedia.org/wiki/RJ45"

Commit message: Mise à jour Régis
Parts:
- J3: symbol e-p-wifi-lf-rescue:RJ45-e-p-wifi-cache-e-p-wifi-lf-rescue -> e-p-wifi-lf-rescue:RJ45-e-p-wifi-cache-e-p-wifi-lf-rescue-e-p-wifi-lf-rescue
Connections:
- net at J2.A3 (Pin_5): now also J3.7_cde_rel; no longer J3.7_itc
- net at J2.A5 (Pin_7): now also J3.8_itc; no longer J3.8_cde_rel
Changed lines of the file:
@@
 	2550 2050 2550 2600
 $Comp
-L e-p-wifi-lf-rescue:RJ45-e-p-wifi-cache-e-p-wifi-lf-rescue J3
+L e-p-wifi-lf-rescue:RJ45-e-p-wifi-cache-e-p-wifi-lf-rescue-e-p-wifi-lf-rescue J3
 U 1 1 62075E51
 P 3450 2250
