File: kicad/e-r-wifi/e-r-wifi-lf/e-r-wifi-lf.kicad_pcb (KiCad board)
At the start: 2 copper layers, 71.8 x 35.6 mm, 8 parts, among them J1 RJ45_conrad_922647, J2 Cde relais, J3 itc, J4 P230V, J5 +5V, J6 Reset, J7 3.3V, SW1 Reset

Commit message: Mise à jour Régis
Parts:
- J2: value Cde relais -> itc
- J3: value itc -> cde relais
Changed lines of the file:
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@@
     (visible_elements FFFFFF7F)
     (pcbplotparams
-      (layerselection 0x010ff_fffffffe)
+      (layerselection 0x01000_fffffffe)
       (usegerberextensions false)
       (usegerberattributes true)
@@
       (padsonsilk false)
       (subtractmaskfromsilk false)
-      (outputformat 1)
+      (outputformat 4)
       (mirror false)
       (drillshape 0)
       (scaleselection 1)
-      (outputdirectory ""))
+      (outputdirectory "/media/airel/SAUV/kicad/"))
   )
   (net 0 "")
@@
       (effects (font (size 1 1) (thickness 0.15)))
     )
-    (fp_text value "Cde relais" (at 4.953 0.889) (layer F.Fab)
+    (fp_text value itc (at 4.826 1.143) (layer F.Fab)
       (effects (font (size 1.15 1.25) (thickness 0.25)))
     )
@@
       (effects (font (size 1 1) (thickness 0.15)))
     )
-    (fp_text value itc (at 4.953 0.508) (layer F.Fab)
-      (effects (font (size 2 2) (thickness 0.25)))
+    (fp_text value "cde relais" (at 4.826 1.651) (layer F.Fab)
+      (effects (font (size 1 1) (thickness 0.25)))
     )
     (fp_line (start 1.8 -1.8) (end -1.8 -1.8) (layer F.CrtYd) (width 0.05))

Commit message: Mise à jour Régis
Other:
- board text added: "e-r-wifi-lf"

Commit message: mise à jour Régis
Other:
- net class Default removed
