File: kicad/e-p-filaire/e-p-wifi.kicad_sch (KiCad schematic)
At the start: 26 parts, among them J1 T1, J2 T2, J3 Masse T1, J4 Conn_02x14_MKR1010, J5 RJ45, Q1 2N2222A

Commit message: Mise à jour Régis
Parts:
- removed J3: Masse T1, Connector_PinHeader_2.54mm:PinHeader_1x02_P2.54mm_Vertical, symbol e-p-wifi-rescue:Conn_01x02-Connector_Generic
- removed R2: 4.7k, Resistor_THT:R_Axial_DIN0207_L6.3mm_D2.5mm_P7.62mm_Horizontal, symbol e-p-wifi-rescue:R-Device
- J2: value T2 -> Nu
- renumbered J4 to J3, J5 to J4, R11 to R10, R12 to R11, R3 to R2, R4 to R3, R5 to R4, R6 to R5, R7 to R6, R8 to R7, R9 to R8, R10 to R9
Connections:
- net GND: now also J2.2 (Pin_2)
- net at J3.D0 (Pin_9): no longer J2.2 (Pin_2)
- no-connect marks 12 -> 13
Other:
- note added: "Interface du thermomètre digital"
- note added: "SCAO/kicad/e-p-filaire/e-p-wifi.kicad_sch"
- note added: "Schéma électrique"
- note added: "Shield MKR wifi 1010 Version filaire"
- note removed: "+5V"
- note removed: "Interface des thermomètres digitaux"
- note removed: "Shield MKR wifi 1010"
- note removed: "T2 -> D0"
- title: Shield du MKR wifi 1010 -> Shield du MKR wifi 1010 - Version filaire
